Commit message: Clearance gate: 1000/1000 doors clear both gates; README quality-gates section + post-mortem; task board
Co-Authored-By: Claude Fable 5.1 <noreply@anthropic.com>

File: assets/doors/db0079_sliding_single/door.urdf (robot description, URDF)
Before this commit: robot db0079_sliding_single_full, 2 links, 1 joints
Links:
- link leaf: mass 51.763028 -> 51.762812; geometry collision box size=1.067 0.044 2.134; collision cylinder length=0.26 radius=0.006

File: assets/doors/db0079_sliding_single/door_simple.urdf (robot description, URDF)
Before this commit: robot db0079_sliding_single_simple, 2 links, 1 joints
Links:
- link leaf: mass 51.760694 -> 51.760478; geometry collision box size=1.067 0.044 2.134; collision cylinder length=0.26 radius=0.006

File: assets/doors/db0095_dutch/door.urdf (robot description, URDF)
Before this commit: robot db0095_dutch_full, 7 links, 6 joints
Links:
- link leaf_lower: mass 1.84692 -> 1.846488; geometry collision box size=0.01 0.024 0.04; collision box size=0.01 0.024 0.04
- link leaf_upper: mass 0.665847 -> 0.665415; geometry collision box size=0.813 0.044 1.17; visual box size=0.004 0.046 1.15

File: assets/doors/db0095_dutch/door_simple.urdf (robot description, URDF)
Before this commit: robot db0095_dutch_simple, 7 links, 6 joints
Links:
- link leaf_lower: mass 1.84624 -> 1.845808; geometry collision box size=0.01 0.024 0.04; collision box size=0.01 0.024 0.04
- link leaf_upper: mass 0.665001 -> 0.664569; geometry collision box size=0.813 0.044 1.17; visual box size=0.753 0.02 0.09

File: assets/doors/db0096_swing_single/door.urdf (robot description, URDF)
Before this commit: robot db0096_swing_single_full, 3 links, 2 joints
Links:
- link leaf: mass 28.411917 -> 28.411485; geometry collision box size=0.762 0.044 2.032; collision cylinder length=0.1 radius=0.008

File: assets/doors/db0096_swing_single/door_simple.urdf (robot description, URDF)
Before this commit: robot db0096_swing_single_simple, 3 links, 2 joints
Links:
- link leaf: mass 28.410436 -> 28.410004; geometry collision box size=0.762 0.044 2.032; collision cylinder length=0.1 radius=0.008

File: assets/doors/db0098_gate_swing/door.urdf (robot description, URDF)
Before this commit: robot db0098_gate_swing_full, 2 links, 1 joints
Links:
- link leaf: mass 14.669311 -> 14.668879; geometry collision box size=1.2 0.025 1.2; collision cylinder length=0.1 radius=0.008

File: assets/doors/db0098_gate_swing/door_simple.urdf (robot description, URDF)
Before this commit: robot db0098_gate_swing_simple, 2 links, 1 joints
Links:
- link leaf: mass 14.668419 -> 14.667987; geometry collision box size=1.2 0.025 1.2; collision cylinder length=0.1 radius=0.008

File: assets/doors/db0127_swing_double/door.urdf (robot description, URDF)
Before this commit: robot db0127_swing_double_full, 4 links, 3 joints
Links:
- link leaf_a: mass 47.339254 -> 47.339038; geometry collision box size=0.9 0.044 2.2; collision cylinder length=0.26 radius=0.006
- link leaf_b: mass 46.356561 -> 46.356345; geometry collision box size=0.021 0.016 0.022; collision box size=0.03 0.006 0.022

File: assets/doors/db0127_swing_double/door_simple.urdf (robot description, URDF)
Before this commit: robot db0127_swing_double_simple, 4 links, 3 joints
Links:
- link leaf_a: mass 47.337249 -> 47.337033; geometry collision box size=0.9 0.044 2.2; collision cylinder length=0.26 radius=0.006
- link leaf_b: mass 46.354555 -> 46.354339; geometry collision box size=0.021 0.016 0.022; collision box size=0.03 0.006 0.022

File: assets/doors/db0134_sliding_single/door.urdf (robot description, URDF)
Before this commit: robot db0134_sliding_single_full, 3 links, 2 joints
Links:
- link leaf: mass 58.190937 -> 58.190505; geometry collision box size=0.813 0.044 2.032; collision cylinder length=0.26 radius=0.006

File: assets/doors/db0134_sliding_single/door_simple.urdf (robot description, URDF)
Before this commit: robot db0134_sliding_single_simple, 3 links, 2 joints
Links:
- link leaf: mass 58.189456 -> 58.189024; geometry collision box size=0.813 0.044 2.032; collision cylinder length=0.26 radius=0.006

File: assets/doors/db0144_swing_double/door.urdf (robot description, URDF)
Before this commit: robot db0144_swing_double_full, 3 links, 2 joints
Links:
- link leaf_a: mass 33.575027 -> 33.574811; geometry collision box size=1 0.044 2; collision cylinder length=0.26 radius=0.006
- link leaf_b: mass 32.586767 -> 32.586551; geometry collision box size=1 0.044 2; visual box size=0.004 0.046 1.98

File: assets/doors/db0144_swing_double/door_simple.urdf (robot description, URDF)
Before this commit: robot db0144_swing_double_simple, 3 links, 2 joints
Links:
- link leaf_a: mass 33.572841 -> 33.572625; geometry collision box size=1 0.044 2; collision cylinder length=0.26 radius=0.006
- link leaf_b: mass 32.584581 -> 32.584365; geometry collision box size=1 0.044 2; visual box size=0.94 0.02 0.09

File: assets/doors/db0151_sliding_single/door.urdf (robot description, URDF)
Before this commit: robot db0151_sliding_single_full, 5 links, 4 joints
Links:
- link leaf: mass 44.866243 -> 44.866027; geometry collision box size=0.914 0.044 2.134; collision cylinder length=0.26 radius=0.006

File: assets/doors/db0151_sliding_single/door_simple.urdf (robot description, URDF)
Before this commit: robot db0151_sliding_single_simple, 5 links, 4 joints
Links:
- link leaf: mass 44.864298 -> 44.864082; geometry collision box size=0.914 0.044 2.134; collision cylinder length=0.26 radius=0.006

File: assets/doors/db0167_sliding_single/door.urdf (robot description, URDF)
Before this commit: robot db0167_sliding_single_full, 2 links, 1 joints
Links:
- link leaf: mass 124.289563 -> 124.289131; geometry collision box size=1.067 0.006 2.4; collision cylinder length=0.26 radius=0.006

File: assets/doors/db0167_sliding_single/door_simple.urdf (robot description, URDF)
Before this commit: robot db0167_sliding_single_simple, 2 links, 1 joints
Links:
- link leaf: mass 124.289106 -> 124.288674; geometry collision box size=1.067 0.006 2.4; collision cylinder length=0.26 radius=0.006

File: assets/doors/db0243_swing_single/door.urdf (robot description, URDF)
Before this commit: robot db0243_swing_single_full, 4 links, 3 joints
Links:
- link leaf: mass 53.489512 -> 53.48908; geometry collision box size=0.813 0.044 2.032; collision cylinder length=0.18 radius=0.008

File: assets/doors/db0243_swing_single/door_simple.urdf (robot description, URDF)
Before this commit: robot db0243_swing_single_simple, 4 links, 3 joints
Links:
- link leaf: mass 53.468046 -> 53.467614; geometry collision box size=0.813 0.044 2.032; collision cylinder length=0.18 radius=0.008
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