Commit message: Regenerate dataset on master (Codex's sliding-track / rising-closer geometry + new QA checks were committed without assets)
Co-Authored-By: Claude Fable 5.1 <noreply@anthropic.com>

File: assets/doors/db0007_sliding_single/door.urdf (robot description, URDF)
Before this commit: robot db0007_sliding_single_full, 2 links, 1 joints
Links:
- link leaf: geometry collision box size=0.914 0.044 2.134; collision cylinder length=0.16 radius=0.0095
- link world_env: geometry collision box size=0.019 0.145 2.154; collision box size=0.024 0.032 0.054

File: assets/doors/db0007_sliding_single/door_simple.urdf (robot description, URDF)
Before this commit: robot db0007_sliding_single_simple, 2 links, 1 joints
Links:
- link leaf: geometry collision box size=0.914 0.044 2.134; collision cylinder length=0.16 radius=0.0095
- link world_env: geometry collision box size=0.019 0.145 2.154; collision box size=0.024 0.032 0.054

File: assets/doors/db0008_sliding_bypass/door.urdf (robot description, URDF)
Before this commit: robot db0008_sliding_bypass_full, 4 links, 3 joints
Links:
- link world_env: geometry collision box size=0.019 0.145 2.052; collision box size=0.056 0.008 0.02

File: assets/doors/db0008_sliding_bypass/door_simple.urdf (robot description, URDF)
Before this commit: robot db0008_sliding_bypass_simple, 4 links, 3 joints
Links:
- link world_env: geometry collision box size=0.019 0.145 2.052; collision box size=0.056 0.008 0.02

File: assets/doors/db0018_sliding_single/door.urdf (robot description, URDF)
Before this commit: robot db0018_sliding_single_full, 2 links, 1 joints
Links:
- link world_env: geometry collision box size=0.079 0.145 2.052; collision box size=0.812 0.016 2.7

File: assets/doors/db0018_sliding_single/door_simple.urdf (robot description, URDF)
Before this commit: robot db0018_sliding_single_simple, 2 links, 1 joints
Links:
- link world_env: geometry collision box size=0.079 0.145 2.052; collision box size=0.812 0.016 2.7

File: assets/doors/db0020_sliding_bypass/door.urdf (robot description, URDF)
Before this commit: robot db0020_sliding_bypass_full, 3 links, 2 joints
Links:
- link world_env: geometry collision box size=0.019 0.145 2.052; collision box size=0.056 0.008 0.02

File: assets/doors/db0020_sliding_bypass/door_simple.urdf (robot description, URDF)
Before this commit: robot db0020_sliding_bypass_simple, 3 links, 2 joints
Links:
- link world_env: geometry collision box size=0.019 0.145 2.052; collision box size=0.056 0.008 0.02

File: assets/doors/db0023_sliding_single/door.urdf (robot description, URDF)
Before this commit: robot db0023_sliding_single_full, 4 links, 3 joints
Links:
- link world_env: geometry collision box size=0.008 0.057 0.12; collision box size=0.016 0.03 0.012

File: assets/doors/db0023_sliding_single/door_minimal.urdf (robot description, URDF)
Before this commit: robot db0023_sliding_single_minimal, 4 links, 3 joints
Links:
- link world_env: geometry collision box size=0.008 0.057 0.12; collision box size=0.016 0.03 0.012

File: assets/doors/db0023_sliding_single/door_simple.urdf (robot description, URDF)
Before this commit: robot db0023_sliding_single_simple, 4 links, 3 joints
Links:
- link world_env: geometry collision box size=0.008 0.057 0.12; collision box size=0.016 0.03 0.012

File: assets/doors/db0029_sliding_single/door.urdf (robot description, URDF)
Before this commit: robot db0029_sliding_single_full, 2 links, 1 joints
Links:
- link leaf: geometry collision box size=1.219 0.044 2.4; collision cylinder length=0.26 radius=0.006
- link world_env: geometry collision box size=0.019 0.145 2.42; collision box size=0.024 0.032 0.054

File: assets/doors/db0029_sliding_single/door_simple.urdf (robot description, URDF)
Before this commit: robot db0029_sliding_single_simple, 2 links, 1 joints
Links:
- link leaf: geometry collision box size=1.219 0.044 2.4; collision cylinder length=0.26 radius=0.006
- link world_env: geometry collision box size=0.019 0.145 2.42; collision box size=0.024 0.032 0.054

File: assets/doors/db0032_sliding_single/door.urdf (robot description, URDF)
Before this commit: robot db0032_sliding_single_full, 4 links, 3 joints
Links:
- link world_env: geometry collision box size=0.008 0.057 0.12; collision box size=0.016 0.03 0.012

File: assets/doors/db0032_sliding_single/door_minimal.urdf (robot description, URDF)
Before this commit: robot db0032_sliding_single_minimal, 4 links, 3 joints
Links:
- link world_env: geometry collision box size=0.008 0.057 0.12; collision box size=0.016 0.03 0.012

File: assets/doors/db0032_sliding_single/door_simple.urdf (robot description, URDF)
Before this commit: robot db0032_sliding_single_simple, 4 links, 3 joints
Links:
- link world_env: geometry collision box size=0.008 0.057 0.12; collision box size=0.016 0.03 0.012

File: assets/doors/db0033_gate_sliding/door.urdf (robot description, URDF)
Before this commit: robot db0033_gate_sliding_full, 3 links, 2 joints
Links:
- link world_env: geometry collision box size=0.008 0.04 0.04; collision box size=0.008 0.04 0.04

File: assets/doors/db0033_gate_sliding/door_minimal.urdf (robot description, URDF)
Before this commit: robot db0033_gate_sliding_minimal, 3 links, 2 joints
Links:
- link world_env: geometry collision box size=0.008 0.04 0.04; collision box size=0.008 0.04 0.04

File: assets/doors/db0033_gate_sliding/door_simple.urdf (robot description, URDF)
Before this commit: robot db0033_gate_sliding_simple, 3 links, 2 joints
Links:
- link world_env: geometry collision box size=0.008 0.04 0.04; collision box size=0.008 0.04 0.04

File: assets/doors/db0038_sliding_single/door.urdf (robot description, URDF)
Before this commit: robot db0038_sliding_single_full, 2 links, 1 joints
Links:
- link world_env: geometry collision box size=0.045 0.145 2.154; collision box size=0.105 0.145 2.154
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