Commit message: Regenerate dataset with the accordion folding mechanism + revolving header clearance fixes (free_opens / no_jam / coupling-range gates)
Co-Authored-By: Claude Fable 5.1 <noreply@anthropic.com>

File: assets/doors/db0004_bifold/door.urdf (robot description, URDF)
Before this commit: robot db0004_bifold_full, 3 links, 2 joints
Links:
- link panel_0_0: mass 7.154123 -> 7.098194; geometry collision box size=0.755 0.035 2.4; visual box size=0.575 0.004 0.05292
- link panel_0_1: mass 7.157637 -> 7.213566; geometry collision box size=0.765 0.035 2.4; collision sphere radius=0.016
- link world_env: geometry collision box size=0.019 0.145 2.455; collision box size=0.019 0.145 2.455
Joints:
- joint panel_0_0_hinge: limit lower=0 upper=1.570796 effort=2000 velocity=10 -> lower=0 upper=1.48353 effort=2000 velocity=10; origin xyz=-0.732 0 0 rpy=0 0 0 -> xyz=-0.7325 0 0 rpy=0 0 0
- joint panel_0_1_hinge: origin xyz=0.727 0 0 rpy=0 0 0 -> xyz=0.727 0.0175 0 rpy=0 0 0

File: assets/doors/db0004_bifold/door_minimal.urdf (robot description, URDF)
Before this commit: robot db0004_bifold_minimal, 3 links, 2 joints
Links:
- link panel_0_0: mass 7.154123 -> 7.098194; geometry collision box size=0.755 0.035 2.4; visual box size=0.755 0.035 2.4
- link panel_0_1: mass 7.157637 -> 7.213566; geometry collision box size=0.765 0.035 2.4; collision sphere radius=0.016
- link world_env: geometry collision box size=0.019 0.145 2.455; collision box size=0.019 0.145 2.455
Joints:
- joint panel_0_0_hinge: limit lower=0 upper=1.570796 effort=2000 velocity=10 -> lower=0 upper=1.48353 effort=2000 velocity=10; origin xyz=-0.732 0 0 rpy=0 0 0 -> xyz=-0.7325 0 0 rpy=0 0 0
- joint panel_0_1_hinge: origin xyz=0.727 0 0 rpy=0 0 0 -> xyz=0.727 0.0175 0 rpy=0 0 0

File: assets/doors/db0004_bifold/door_simple.urdf (robot description, URDF)
Before this commit: robot db0004_bifold_simple, 3 links, 2 joints
Links:
- link panel_0_0: mass 7.154123 -> 7.098194; geometry collision box size=0.755 0.035 2.4; visual box size=0.755 0.035 2.4
- link panel_0_1: mass 7.157637 -> 7.213566; geometry collision box size=0.765 0.035 2.4; collision sphere radius=0.016
- link world_env: geometry collision box size=0.019 0.145 2.455; collision box size=0.019 0.145 2.455
Joints:
- joint panel_0_0_hinge: limit lower=0 upper=1.570796 effort=2000 velocity=10 -> lower=0 upper=1.48353 effort=2000 velocity=10; origin xyz=-0.732 0 0 rpy=0 0 0 -> xyz=-0.7325 0 0 rpy=0 0 0
- joint panel_0_1_hinge: origin xyz=0.727 0 0 rpy=0 0 0 -> xyz=0.727 0.0175 0 rpy=0 0 0

File: assets/doors/db0009_bifold/door.urdf (robot description, URDF)
Before this commit: robot db0009_bifold_full, 5 links, 4 joints
Links:
- link panel_0_0: mass 1.407017 -> 1.36296; geometry collision box size=0.183 0.035 2.032; visual box size=0.183 0.035 2.032
- link panel_0_1: mass 1.410543 -> 1.4546; geometry collision box size=0.193028 0.035 2.032; collision sphere radius=0.016
- link panel_1_0: mass 1.407017 -> 1.36296; geometry collision box size=0.183 0.035 2.032; visual box size=0.183 0.035 2.032
- link panel_1_1: mass 1.410543 -> 1.4546; geometry collision box size=0.193028 0.035 2.032; collision sphere radius=0.016
- link world_env: geometry collision box size=0.019 0.145 2.087; collision box size=0.019 0.145 2.087
Joints:
- joint panel_0_0_hinge: limit lower=0 upper=1.570796 effort=2000 velocity=10 -> lower=0 upper=1.48353 effort=2000 velocity=10; origin xyz=-0.351 0 0 rpy=0 0 0 -> xyz=-0.356 0 0 rpy=0 0 0
- joint panel_0_1_hinge: origin xyz=0.155 0 0 rpy=0 0 0 -> xyz=0.155 0.0175 0 rpy=0 0 0
- joint panel_1_0_hinge: limit lower=0 upper=1.570796 effort=2000 velocity=10 -> lower=0 upper=1.48353 effort=2000 velocity=10; origin xyz=0.351 0 0 rpy=0 0 0 -> xyz=0.356 0 0 rpy=0 0 0
- joint panel_1_1_hinge: origin xyz=-0.155 0 0 rpy=0 0 0 -> xyz=-0.155 0.0175 0 rpy=0 0 0

File: assets/doors/db0009_bifold/door_minimal.urdf (robot description, URDF)
Before this commit: robot db0009_bifold_minimal, 5 links, 4 joints
Links:
- link panel_0_0: mass 1.407017 -> 1.36296; geometry collision box size=0.183 0.035 2.032; visual box size=0.183 0.035 2.032
- link panel_0_1: mass 1.410543 -> 1.4546; geometry collision box size=0.193028 0.035 2.032; collision sphere radius=0.016
- link panel_1_0: mass 1.407017 -> 1.36296; geometry collision box size=0.183 0.035 2.032; visual box size=0.183 0.035 2.032
- link panel_1_1: mass 1.410543 -> 1.4546; geometry collision box size=0.193028 0.035 2.032; collision sphere radius=0.016
- link world_env: geometry collision box size=0.019 0.145 2.087; collision box size=0.019 0.145 2.087
Joints:
- joint panel_0_0_hinge: limit lower=0 upper=1.570796 effort=2000 velocity=10 -> lower=0 upper=1.48353 effort=2000 velocity=10; origin xyz=-0.351 0 0 rpy=0 0 0 -> xyz=-0.356 0 0 rpy=0 0 0
- joint panel_0_1_hinge: origin xyz=0.155 0 0 rpy=0 0 0 -> xyz=0.155 0.0175 0 rpy=0 0 0
- joint panel_1_0_hinge: limit lower=0 upper=1.570796 effort=2000 velocity=10 -> lower=0 upper=1.48353 effort=2000 velocity=10; origin xyz=0.351 0 0 rpy=0 0 0 -> xyz=0.356 0 0 rpy=0 0 0
- joint panel_1_1_hinge: origin xyz=-0.155 0 0 rpy=0 0 0 -> xyz=-0.155 0.0175 0 rpy=0 0 0

File: assets/doors/db0009_bifold/door_simple.urdf (robot description, URDF)
Before this commit: robot db0009_bifold_simple, 5 links, 4 joints
Links:
- link panel_0_0: mass 1.407017 -> 1.36296; geometry collision box size=0.183 0.035 2.032; visual box size=0.183 0.035 2.032
- link panel_0_1: mass 1.410543 -> 1.4546; geometry collision box size=0.193028 0.035 2.032; collision sphere radius=0.016
- link panel_1_0: mass 1.407017 -> 1.36296; geometry collision box size=0.183 0.035 2.032; visual box size=0.183 0.035 2.032
- link panel_1_1: mass 1.410543 -> 1.4546; geometry collision box size=0.193028 0.035 2.032; collision sphere radius=0.016
- link world_env: geometry collision box size=0.019 0.145 2.087; collision box size=0.019 0.145 2.087
Joints:
- joint panel_0_0_hinge: limit lower=0 upper=1.570796 effort=2000 velocity=10 -> lower=0 upper=1.48353 effort=2000 velocity=10; origin xyz=-0.351 0 0 rpy=0 0 0 -> xyz=-0.356 0 0 rpy=0 0 0
- joint panel_0_1_hinge: origin xyz=0.155 0 0 rpy=0 0 0 -> xyz=0.155 0.0175 0 rpy=0 0 0
- joint panel_1_0_hinge: limit lower=0 upper=1.570796 effort=2000 velocity=10 -> lower=0 upper=1.48353 effort=2000 velocity=10; origin xyz=0.351 0 0 rpy=0 0 0 -> xyz=0.356 0 0 rpy=0 0 0
- joint panel_1_1_hinge: origin xyz=-0.155 0 0 rpy=0 0 0 -> xyz=-0.155 0.0175 0 rpy=0 0 0

File: assets/doors/db0030_bifold/door.urdf (robot description, URDF)
Before this commit: robot db0030_bifold_full, 3 links, 2 joints
Links:
- link panel_0_0: mass 3.093804 -> 3.044262; geometry collision box size=0.374 0.035 2.032; visual box size=0.194 0.004 0.052712
- link panel_0_1: mass 3.097474 -> 3.147016; geometry collision box size=0.384 0.035 2.032; collision sphere radius=0.016
- link world_env: geometry collision box size=0.019 0.145 2.087; collision box size=0.019 0.145 2.087
Joints:
- joint panel_0_0_hinge: limit lower=0 upper=1.570796 effort=2000 velocity=10 -> lower=0 upper=1.48353 effort=2000 velocity=10; origin xyz=-0.351 0 0 rpy=0 0 0 -> xyz=-0.3515 0 0 rpy=0 0 0
- joint panel_0_1_hinge: origin xyz=0.346 0 0 rpy=0 0 0 -> xyz=0.346 0.0175 0 rpy=0 0 0

File: assets/doors/db0030_bifold/door_minimal.urdf (robot description, URDF)
Before this commit: robot db0030_bifold_minimal, 3 links, 2 joints
Links:
- link panel_0_0: mass 3.093804 -> 3.044262; geometry collision box size=0.374 0.035 2.032; visual box size=0.374 0.035 2.032
- link panel_0_1: mass 3.097474 -> 3.147016; geometry collision box size=0.384 0.035 2.032; collision sphere radius=0.016
- link world_env: geometry collision box size=0.019 0.145 2.087; collision box size=0.019 0.145 2.087
Joints:
- joint panel_0_0_hinge: limit lower=0 upper=1.570796 effort=2000 velocity=10 -> lower=0 upper=1.48353 effort=2000 velocity=10; origin xyz=-0.351 0 0 rpy=0 0 0 -> xyz=-0.3515 0 0 rpy=0 0 0
- joint panel_0_1_hinge: origin xyz=0.346 0 0 rpy=0 0 0 -> xyz=0.346 0.0175 0 rpy=0 0 0

File: assets/doors/db0030_bifold/door_simple.urdf (robot description, URDF)
Before this commit: robot db0030_bifold_simple, 3 links, 2 joints
Links:
- link panel_0_0: mass 3.093804 -> 3.044262; geometry collision box size=0.374 0.035 2.032; visual box size=0.374 0.035 2.032
- link panel_0_1: mass 3.097474 -> 3.147016; geometry collision box size=0.384 0.035 2.032; collision sphere radius=0.016
- link world_env: geometry collision box size=0.019 0.145 2.087; collision box size=0.019 0.145 2.087
Joints:
- joint panel_0_0_hinge: limit lower=0 upper=1.570796 effort=2000 velocity=10 -> lower=0 upper=1.48353 effort=2000 velocity=10; origin xyz=-0.351 0 0 rpy=0 0 0 -> xyz=-0.3515 0 0 rpy=0 0 0
- joint panel_0_1_hinge: origin xyz=0.346 0 0 rpy=0 0 0 -> xyz=0.346 0.0175 0 rpy=0 0 0

File: assets/doors/db0037_strip_curtain/door.urdf (robot description, URDF)
Before this commit: robot db0037_strip_curtain_full, 6 links, 5 joints
Joints:
- joint strip_0_hinge: origin xyz=-0.31 -0.003 2.414 rpy=0 0 0 -> xyz=-0.3 -0.007 2.414 rpy=0 0 0
- joint strip_1_hinge: origin xyz=-0.155 0.003 2.414 rpy=0 0 0 -> xyz=-0.15 0.003 2.414 rpy=0 0 0
- joint strip_2_hinge: origin xyz=0 -0.003 2.414 rpy=0 0 0 -> xyz=0 0.001 2.414 rpy=0 0 0
- joint strip_3_hinge: origin xyz=0.155 0.003 2.414 rpy=0 0 0 -> xyz=0.15 -0.001 2.414 rpy=0 0 0
- joint strip_4_hinge: origin xyz=0.31 -0.003 2.414 rpy=0 0 0 -> xyz=0.3 -0.003 2.414 rpy=0 0 0

File: assets/doors/db0037_strip_curtain/door_minimal.urdf (robot description, URDF)
Before this commit: robot db0037_strip_curtain_minimal, 4 links, 3 joints
Joints:
- joint strip_0_hinge: origin xyz=-0.31 -0.003 2.414 rpy=0 0 0 -> xyz=-0.3 -0.007 2.414 rpy=0 0 0
- joint strip_2_hinge: origin xyz=0 -0.003 2.414 rpy=0 0 0 -> xyz=0 0.001 2.414 rpy=0 0 0
- joint strip_4_hinge: origin xyz=0.31 -0.003 2.414 rpy=0 0 0 -> xyz=0.3 -0.003 2.414 rpy=0 0 0

File: assets/doors/db0037_strip_curtain/door_simple.urdf (robot description, URDF)
Before this commit: robot db0037_strip_curtain_simple, 6 links, 5 joints
Joints:
- joint strip_0_hinge: origin xyz=-0.31 -0.003 2.414 rpy=0 0 0 -> xyz=-0.3 -0.007 2.414 rpy=0 0 0
- joint strip_1_hinge: origin xyz=-0.155 0.003 2.414 rpy=0 0 0 -> xyz=-0.15 0.003 2.414 rpy=0 0 0
- joint strip_2_hinge: origin xyz=0 -0.003 2.414 rpy=0 0 0 -> xyz=0 0.001 2.414 rpy=0 0 0
- joint strip_3_hinge: origin xyz=0.155 0.003 2.414 rpy=0 0 0 -> xyz=0.15 -0.001 2.414 rpy=0 0 0
- joint strip_4_hinge: origin xyz=0.31 -0.003 2.414 rpy=0 0 0 -> xyz=0.3 -0.003 2.414 rpy=0 0 0

File: assets/doors/db0043_bifold/door.urdf (robot description, URDF)
Before this commit: robot db0043_bifold_full, 3 links, 2 joints
Links:
- link panel_0_0: mass 3.676531 -> 3.625049; geometry collision box size=0.45 0.035 2.032; visual box size=0.23 0.006 1.66688
- link panel_0_1: mass 3.691327 -> 3.742809; geometry collision box size=0.46 0.035 2.032; collision cylinder length=0.16 radius=0.0095
- link world_env: geometry collision box size=0.019 0.145 2.087; collision box size=0.019 0.145 2.087
Joints:
- joint panel_0_0_hinge: limit lower=0 upper=1.570796 effort=2000 velocity=10 -> lower=0 upper=1.48353 effort=2000 velocity=10; origin xyz=-0.427 0 0 rpy=0 0 0 -> xyz=-0.4275 0 0 rpy=0 0 0
- joint panel_0_1_hinge: origin xyz=0.422 0 0 rpy=0 0 0 -> xyz=0.422 0.0175 0 rpy=0 0 0

File: assets/doors/db0043_bifold/door_minimal.urdf (robot description, URDF)
Before this commit: robot db0043_bifold_minimal, 3 links, 2 joints
Links:
- link panel_0_0: mass 3.676531 -> 3.625049; geometry collision box size=0.45 0.035 2.032; visual box size=0.45 0.035 2.032
- link panel_0_1: mass 3.691327 -> 3.742809; geometry collision box size=0.46 0.035 2.032; collision cylinder length=0.16 radius=0.0095
- link world_env: geometry collision box size=0.019 0.145 2.087; collision box size=0.019 0.145 2.087
Joints:
- joint panel_0_0_hinge: limit lower=0 upper=1.570796 effort=2000 velocity=10 -> lower=0 upper=1.48353 effort=2000 velocity=10; origin xyz=-0.427 0 0 rpy=0 0 0 -> xyz=-0.4275 0 0 rpy=0 0 0
- joint panel_0_1_hinge: origin xyz=0.422 0 0 rpy=0 0 0 -> xyz=0.422 0.0175 0 rpy=0 0 0

File: assets/doors/db0043_bifold/door_simple.urdf (robot description, URDF)
Before this commit: robot db0043_bifold_simple, 3 links, 2 joints
Links:
- link panel_0_0: mass 3.676531 -> 3.625049; geometry collision box size=0.45 0.035 2.032; visual box size=0.23 0.006 1.66688
- link panel_0_1: mass 3.691327 -> 3.742809; geometry collision box size=0.46 0.035 2.032; collision cylinder length=0.16 radius=0.0095
- link world_env: geometry collision box size=0.019 0.145 2.087; collision box size=0.019 0.145 2.087
Joints:
- joint panel_0_0_hinge: limit lower=0 upper=1.570796 effort=2000 velocity=10 -> lower=0 upper=1.48353 effort=2000 velocity=10; origin xyz=-0.427 0 0 rpy=0 0 0 -> xyz=-0.4275 0 0 rpy=0 0 0
- joint panel_0_1_hinge: origin xyz=0.422 0 0 rpy=0 0 0 -> xyz=0.422 0.0175 0 rpy=0 0 0

File: assets/doors/db0045_pet_door/door.urdf (robot description, URDF)
Before this commit: robot db0045_pet_door_full, 2 links, 1 joints
Joints:
- joint flap_hinge: origin xyz=0 0 0.56 rpy=0 0 0 -> xyz=0 0 0.5535 rpy=0 0 0

File: assets/doors/db0045_pet_door/door_minimal.urdf (robot description, URDF)
Before this commit: robot db0045_pet_door_minimal, 2 links, 1 joints
Joints:
- joint flap_hinge: origin xyz=0 0 0.56 rpy=0 0 0 -> xyz=0 0 0.5535 rpy=0 0 0

File: assets/doors/db0045_pet_door/door_simple.urdf (robot description, URDF)
Before this commit: robot db0045_pet_door_simple, 2 links, 1 joints
Joints:
- joint flap_hinge: origin xyz=0 0 0.56 rpy=0 0 0 -> xyz=0 0 0.5535 rpy=0 0 0

File: assets/doors/db0052_pet_door/door.urdf (robot description, URDF)
Before this commit: robot db0052_pet_door_full, 2 links, 1 joints
Joints:
- joint flap_hinge: origin xyz=0 0 0.44 rpy=0 0 0 -> xyz=0 0 0.434 rpy=0 0 0

File: assets/doors/db0052_pet_door/door_minimal.urdf (robot description, URDF)
Before this commit: robot db0052_pet_door_minimal, 2 links, 1 joints
Joints:
- joint flap_hinge: origin xyz=0 0 0.44 rpy=0 0 0 -> xyz=0 0 0.434 rpy=0 0 0
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