Commit message: Deterministic kinematic clearance gate + geometry fixes: 1000/1000 doors clear
- doorbench/clearance.py: sweeps every joint of every door with ALL geometry collidable (visual parts included) and
  parent-child filtering disabled; any interpenetration > 2 mm fails; wired into qa.json (checks.clearance) and manifest
- scripts/clearance_report.py: dataset-wide grouped report
- fixes found by the gate: butt hinges rebuilt (both plates in the edge/jamb plane, jamb plate static), closer arms above
  the head with the shoe on the casing, exit-device housings as convex primitives + pad clearance + vertical rods inside
  the leaf, mullions via strike columns with ramps, roll-up coil/hood off the curtain path, garage C-channel tracks,
  strip curtains staggered in 3 layers, lever escutcheons static, keypad/thumbturn on opposite faces, maglocks on the
  stop side, vault crane hinges outside the wall, tripod housing recess, saloon/baby-gate centre pivots with proper
  gaps, double-egress thin partition, single-slide auto door layout, pet-flap holes cut out of the slab, and
  opening-angle caps by casing/closer/strap/brace
- TASKS.md task board

Co-Authored-By: Claude Fable 5.1 <noreply@anthropic.com>

File: assets/doors/db0001_rollup/door.urdf (robot description, URDF)
Before this commit: robot db0001_rollup_full, 2 links, 1 joints
Links:
- link world_env: geometry collision box size=0.06 0.05 2.49; collision box size=0.06 0.05 2.49

File: assets/doors/db0001_rollup/door_simple.urdf (robot description, URDF)
Before this commit: robot db0001_rollup_simple, 2 links, 1 joints
Links:
- link world_env: geometry collision box size=0.06 0.05 2.49; collision box size=0.06 0.05 2.49

File: assets/doors/db0002_swing_single/door.urdf (robot description, URDF)
Before this commit: robot db0002_swing_single_full, 5 links, 4 joints
Links:
- link leaf: mass 12.035386 -> 11.747998; geometry collision box size=0.762 0.035 2.0216; visual box size=0.542 0.006 0.764072
- link leaf_handle: mass 1.133308 -> 1.127981; geometry collision cylinder length=0.024 radius=0.011; collision cylinder length=0.024 radius=0.011
- link world_env: geometry collision box size=0.011 0.032 2.045; collision box size=0.011 0.032 2.045

File: assets/doors/db0002_swing_single/door_simple.urdf (robot description, URDF)
Before this commit: robot db0002_swing_single_simple, 5 links, 4 joints
Links:
- link leaf: mass 12.035386 -> 11.747998; geometry collision box size=0.762 0.035 2.0216; visual box size=0.542 0.006 0.764072
- link world_env: geometry collision box size=0.011 0.032 2.045; collision box size=0.011 0.032 2.045

File: assets/doors/db0003_cold_storage/door.urdf (robot description, URDF)
Before this commit: robot db0003_cold_storage_full, 5 links, 4 joints
Links:
- link leaf: mass 46.18519 -> 45.727378
- link leaf_handle: mass 2.977173 -> 2.971846; geometry collision cylinder length=0.044 radius=0.012; collision cylinder length=0.044 radius=0.012
- link world_env: geometry collision box size=0.011 0.032 2.15; collision box size=0.011 0.032 2.15

File: assets/doors/db0003_cold_storage/door_simple.urdf (robot description, URDF)
Before this commit: robot db0003_cold_storage_simple, 5 links, 4 joints
Links:
- link leaf: mass 46.11479 -> 45.656978
- link world_env: geometry collision box size=0.011 0.032 2.15; collision box size=0.011 0.032 2.15

File: assets/doors/db0004_bifold/door.urdf (robot description, URDF)
Before this commit: robot db0004_bifold_full, 3 links, 2 joints
Joints:
- joint panel_0_0_hinge: origin xyz=-0.747 0 0 rpy=0 0 0 -> xyz=-0.732 0 0 rpy=0 0 0
- joint panel_0_1_hinge: origin xyz=0.742 0 0 rpy=0 0 0 -> xyz=0.727 0 0 rpy=0 0 0

File: assets/doors/db0004_bifold/door_minimal.urdf (robot description, URDF)
Before this commit: robot db0004_bifold_minimal, 3 links, 2 joints
Joints:
- joint panel_0_0_hinge: origin xyz=-0.747 0 0 rpy=0 0 0 -> xyz=-0.732 0 0 rpy=0 0 0
- joint panel_0_1_hinge: origin xyz=0.742 0 0 rpy=0 0 0 -> xyz=0.727 0 0 rpy=0 0 0

File: assets/doors/db0004_bifold/door_simple.urdf (robot description, URDF)
Before this commit: robot db0004_bifold_simple, 3 links, 2 joints
Joints:
- joint panel_0_0_hinge: origin xyz=-0.747 0 0 rpy=0 0 0 -> xyz=-0.732 0 0 rpy=0 0 0
- joint panel_0_1_hinge: origin xyz=0.742 0 0 rpy=0 0 0 -> xyz=0.727 0 0 rpy=0 0 0

File: assets/doors/db0006_gate_swing/door.urdf (robot description, URDF)
Before this commit: robot db0006_gate_swing_full, 3 links, 2 joints
Links:
- link leaf: mass 76.958148 -> 76.727436
- link world_env: geometry collision box size=0.03 0.006 0.03; collision box size=0.04 0.024 0.12
Joints:
- joint leaf_hinge: limit lower=0 upper=3.141593 effort=2000 velocity=10 -> lower=0 upper=1.745329 effort=2000 velocity=10

File: assets/doors/db0006_gate_swing/door_minimal.urdf (robot description, URDF)
Before this commit: robot db0006_gate_swing_minimal, 3 links, 2 joints
Links:
- link world_env: geometry collision box size=0.03 0.006 0.03; collision box size=0.04 0.024 0.12
Joints:
- joint leaf_hinge: limit lower=0 upper=3.141593 effort=2000 velocity=10 -> lower=0 upper=1.745329 effort=2000 velocity=10

File: assets/doors/db0006_gate_swing/door_simple.urdf (robot description, URDF)
Before this commit: robot db0006_gate_swing_simple, 3 links, 2 joints
Links:
- link leaf: mass 76.944669 -> 76.713957
- link world_env: geometry collision box size=0.03 0.006 0.03; collision box size=0.04 0.024 0.12
Joints:
- joint leaf_hinge: limit lower=0 upper=3.141593 effort=2000 velocity=10 -> lower=0 upper=1.745329 effort=2000 velocity=10

File: assets/doors/db0007_sliding_single/door.urdf (robot description, URDF)
Before this commit: robot db0007_sliding_single_full, 2 links, 1 joints
Joints:
- joint leaf_slide: origin xyz=0 -0.1075 0 rpy=0 0 0 -> xyz=0 -0.1145 0 rpy=0 0 0

File: assets/doors/db0007_sliding_single/door_minimal.urdf (robot description, URDF)
Before this commit: robot db0007_sliding_single_minimal, 2 links, 1 joints
Joints:
- joint leaf_slide: origin xyz=0 -0.1075 0 rpy=0 0 0 -> xyz=0 -0.1145 0 rpy=0 0 0

File: assets/doors/db0007_sliding_single/door_simple.urdf (robot description, URDF)
Before this commit: robot db0007_sliding_single_simple, 2 links, 1 joints
Joints:
- joint leaf_slide: origin xyz=0 -0.1075 0 rpy=0 0 0 -> xyz=0 -0.1145 0 rpy=0 0 0

File: assets/doors/db0008_sliding_bypass/door.urdf (robot description, URDF)
Before this commit: robot db0008_sliding_bypass_full, 4 links, 3 joints
Links:
- link leaf_0: mass 37.158849 -> 37.158145; geometry collision box size=1.219 0.006 2.032; visual box size=0.055 0.001 0.055
- link leaf_1: mass 37.158849 -> 37.158145; geometry collision box size=1.219 0.006 2.032; visual box size=0.055 0.001 0.055
- link leaf_2: mass 37.158849 -> 37.158145; geometry collision box size=1.219 0.006 2.032; visual box size=0.055 0.001 0.055
Joints:
- joint leaf_0_slide: origin xyz=-1.194 -0.007 0 rpy=0 0 0 -> xyz=-1.194 -0.056 0 rpy=0 0 0
- joint leaf_1_slide: origin xyz=-0.005 0.007 0 rpy=0 0 0 -> xyz=-0.005 0 0 rpy=0 0 0
- joint leaf_2_slide: origin xyz=1.184 -0.007 0 rpy=0 0 0 -> xyz=1.184 0.056 0 rpy=0 0 0

File: assets/doors/db0008_sliding_bypass/door_minimal.urdf (robot description, URDF)
Before this commit: robot db0008_sliding_bypass_minimal, 4 links, 3 joints
Joints:
- joint leaf_0_slide: origin xyz=-1.194 -0.007 0 rpy=0 0 0 -> xyz=-1.194 -0.056 0 rpy=0 0 0
- joint leaf_1_slide: origin xyz=-0.005 0.007 0 rpy=0 0 0 -> xyz=-0.005 0 0 rpy=0 0 0
- joint leaf_2_slide: origin xyz=1.184 -0.007 0 rpy=0 0 0 -> xyz=1.184 0.056 0 rpy=0 0 0

File: assets/doors/db0008_sliding_bypass/door_simple.urdf (robot description, URDF)
Before this commit: robot db0008_sliding_bypass_simple, 4 links, 3 joints
Links:
- link leaf_0: mass 37.158849 -> 37.158145; geometry collision box size=1.219 0.006 2.032; visual box size=0.055 0.001 0.055
- link leaf_1: mass 37.158849 -> 37.158145; geometry collision box size=1.219 0.006 2.032; visual box size=0.055 0.001 0.055
- link leaf_2: mass 37.158849 -> 37.158145; geometry collision box size=1.219 0.006 2.032; visual box size=0.055 0.001 0.055
Joints:
- joint leaf_0_slide: origin xyz=-1.194 -0.007 0 rpy=0 0 0 -> xyz=-1.194 -0.056 0 rpy=0 0 0
- joint leaf_1_slide: origin xyz=-0.005 0.007 0 rpy=0 0 0 -> xyz=-0.005 0 0 rpy=0 0 0
- joint leaf_2_slide: origin xyz=1.184 -0.007 0 rpy=0 0 0 -> xyz=1.184 0.056 0 rpy=0 0 0

File: assets/doors/db0009_bifold/door.urdf (robot description, URDF)
Before this commit: robot db0009_bifold_full, 5 links, 4 joints
Joints:
- joint panel_0_0_hinge: origin xyz=-0.366 0 0 rpy=0 0 0 -> xyz=-0.351 0 0 rpy=0 0 0
- joint panel_0_1_hinge: origin xyz=0.17 0 0 rpy=0 0 0 -> xyz=0.155 0 0 rpy=0 0 0
- joint panel_1_0_hinge: origin xyz=0.366 0 0 rpy=0 0 0 -> xyz=0.351 0 0 rpy=0 0 0
- joint panel_1_1_hinge: origin xyz=-0.17 0 0 rpy=0 0 0 -> xyz=-0.155 0 0 rpy=0 0 0

File: assets/doors/db0009_bifold/door_minimal.urdf (robot description, URDF)
Before this commit: robot db0009_bifold_minimal, 5 links, 4 joints
Joints:
- joint panel_0_0_hinge: origin xyz=-0.366 0 0 rpy=0 0 0 -> xyz=-0.351 0 0 rpy=0 0 0
- joint panel_0_1_hinge: origin xyz=0.17 0 0 rpy=0 0 0 -> xyz=0.155 0 0 rpy=0 0 0
- joint panel_1_0_hinge: origin xyz=0.366 0 0 rpy=0 0 0 -> xyz=0.351 0 0 rpy=0 0 0
- joint panel_1_1_hinge: origin xyz=-0.17 0 0 rpy=0 0 0 -> xyz=-0.155 0 0 rpy=0 0 0
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
Commit message: Mass gate: reconcile every door's moving mass to the derived spec mass (checks.mass); keypad locks require a keypad operator; sectional counterbalance from spec mass
Found by the MuJoCo import agent: 315/1000 doors had simulated masses far from spec (glass panes at token
density, split leaves without a share, strips each carrying the whole curtain, rotors at raw material density).
build.py now distributes (total - modelled hardware) over the leaf bodies by volume; qa.py checks it.
1000/1000 doors pass all gates; 267 tests green.

Co-Authored-By: Claude Fable 5.1 <noreply@anthropic.com>

File: assets/doors/db0001_rollup/door.urdf (robot description, URDF)
Before this commit: robot db0001_rollup_full, 2 links, 1 joints
Links:
- link curtain: mass 45.213516 -> 37.888608

File: assets/doors/db0001_rollup/door_minimal.urdf (robot description, URDF)
Before this commit: robot db0001_rollup_minimal, 2 links, 1 joints
Links:
- link curtain: mass 45.212608 -> 37.888608

File: assets/doors/db0001_rollup/door_simple.urdf (robot description, URDF)
Before this commit: robot db0001_rollup_simple, 2 links, 1 joints
Links:
- link curtain: mass 45.212608 -> 37.888608

File: assets/doors/db0002_swing_single/door.urdf (robot description, URDF)
Before this commit: robot db0002_swing_single_full, 5 links, 4 joints
Links:
- link leaf: mass 11.747998 -> 11.329802

File: assets/doors/db0002_swing_single/door_minimal.urdf (robot description, URDF)
Before this commit: robot db0002_swing_single_minimal, 5 links, 4 joints
Links:
- link leaf: mass 11.151307 -> 11.329802

File: assets/doors/db0002_swing_single/door_simple.urdf (robot description, URDF)
Before this commit: robot db0002_swing_single_simple, 5 links, 4 joints
Links:
- link leaf: mass 11.747998 -> 11.329802

File: assets/doors/db0003_cold_storage/door.urdf (robot description, URDF)
Before this commit: robot db0003_cold_storage_full, 5 links, 4 joints
Links:
- link leaf: mass 45.727378 -> 43.850003

File: assets/doors/db0003_cold_storage/door_minimal.urdf (robot description, URDF)
Before this commit: robot db0003_cold_storage_minimal, 5 links, 4 joints
Links:
- link leaf: mass 41.354717 -> 43.850003

File: assets/doors/db0003_cold_storage/door_simple.urdf (robot description, URDF)
Before this commit: robot db0003_cold_storage_simple, 5 links, 4 joints
Links:
- link leaf: mass 45.656978 -> 43.850003

File: assets/doors/db0004_bifold/door.urdf (robot description, URDF)
Before this commit: robot db0004_bifold_full, 3 links, 2 joints
Links:
- link panel_0_0: mass 14.086688 -> 7.154123
- link panel_0_1: mass 0.1705 -> 7.157637

File: assets/doors/db0004_bifold/door_minimal.urdf (robot description, URDF)
Before this commit: robot db0004_bifold_minimal, 3 links, 2 joints
Links:
- link panel_0_0: mass 14.08176 -> 7.154123
- link panel_0_1: mass 0.165572 -> 7.157637

File: assets/doors/db0004_bifold/door_simple.urdf (robot description, URDF)
Before this commit: robot db0004_bifold_simple, 3 links, 2 joints
Links:
- link panel_0_0: mass 14.08176 -> 7.154123
- link panel_0_1: mass 0.165572 -> 7.157637

File: assets/doors/db0005_garage_tiltup/door.urdf (robot description, URDF)
Before this commit: robot db0005_garage_tiltup_full, 2 links, 1 joints
Links:
- link door: mass 82.366247 -> 83.5559

File: assets/doors/db0005_garage_tiltup/door_minimal.urdf (robot description, URDF)
Before this commit: robot db0005_garage_tiltup_minimal, 2 links, 1 joints
Links:
- link door: mass 82.3599 -> 83.5559

File: assets/doors/db0005_garage_tiltup/door_simple.urdf (robot description, URDF)
Before this commit: robot db0005_garage_tiltup_simple, 2 links, 1 joints
Links:
- link door: mass 82.3599 -> 83.5559

File: assets/doors/db0006_gate_swing/door.urdf (robot description, URDF)
Before this commit: robot db0006_gate_swing_full, 3 links, 2 joints
Links:
- link leaf: mass 76.727436 -> 76.776258

File: assets/doors/db0006_gate_swing/door_minimal.urdf (robot description, URDF)
Before this commit: robot db0006_gate_swing_minimal, 3 links, 2 joints
Links:
- link leaf: mass 75.474 -> 76.776258

File: assets/doors/db0006_gate_swing/door_simple.urdf (robot description, URDF)
Before this commit: robot db0006_gate_swing_simple, 3 links, 2 joints
Links:
- link leaf: mass 76.713957 -> 76.776258

File: assets/doors/db0007_sliding_single/door.urdf (robot description, URDF)
Before this commit: robot db0007_sliding_single_full, 2 links, 1 joints
Links:
- link leaf: mass 63.700369 -> 60.574661

File: assets/doors/db0007_sliding_single/door_minimal.urdf (robot description, URDF)
Before this commit: robot db0007_sliding_single_minimal, 2 links, 1 joints
Links:
- link leaf: mass 60.524302 -> 60.574661
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