Commit message: Round-3 parity fixes: real env-release welds + self-collision + bilateral couplings in USD, protocol/metric corrections with staleness gating, running-clearance gate (139 doors of zero-clearance geometry fixed)
Co-Authored-By: Claude Opus 5 <noreply@anthropic.com>

File: assets/doors/db0001_rollup/door.urdf (robot description, URDF)
Before this commit: robot db0001_rollup_full, 2 links, 1 joints
Links:
- link curtain: geometry collision box size=0.2 0.012 0.03; collision box size=2.44 0.0008 2.44

File: assets/doors/db0001_rollup/door_minimal.urdf (robot description, URDF)
Before this commit: robot db0001_rollup_minimal, 2 links, 1 joints
Links:
- link curtain: geometry collision box size=0.2 0.012 0.03; collision box size=2.44 0.0008 2.44

File: assets/doors/db0001_rollup/door_simple.urdf (robot description, URDF)
Before this commit: robot db0001_rollup_simple, 2 links, 1 joints
Links:
- link curtain: geometry collision box size=0.2 0.012 0.03; collision box size=2.44 0.0008 2.44

File: assets/doors/db0002_swing_single/door.urdf (robot description, URDF)
Before this commit: robot db0002_swing_single_full, 5 links, 4 joints
Links:
- link world_env: geometry collision box size=0.011 0.032 2.045; collision box size=0.011 0.032 2.045

File: assets/doors/db0002_swing_single/door_minimal.urdf (robot description, URDF)
Before this commit: robot db0002_swing_single_minimal, 5 links, 4 joints
Links:
- link world_env: geometry collision box size=0.011 0.032 2.045; collision box size=0.011 0.032 2.045

File: assets/doors/db0002_swing_single/door_simple.urdf (robot description, URDF)
Before this commit: robot db0002_swing_single_simple, 5 links, 4 joints
Links:
- link world_env: geometry collision box size=0.011 0.032 2.045; collision box size=0.011 0.032 2.045

File: assets/doors/db0004_bifold/door.urdf (robot description, URDF)
Before this commit: robot db0004_bifold_full, 3 links, 2 joints
Links:
- link panel_0_0: mass 7.098194 -> 7.061165; geometry collision box size=0.751291 0.035 2.4; visual box size=0.571291 0.004 0.05292
- link panel_0_1: mass 7.213566 -> 7.250595; geometry collision box size=0.769 0.035 2.4; collision sphere radius=0.016
- link world_env: geometry collision box size=0.019 0.145 2.455; collision box size=0.019 0.145 2.455
Joints:
- joint panel_0_0_hinge: origin xyz=-0.7325 0 0 rpy=0 0 0 -> xyz=-0.7345 0 0 rpy=0 0 0

File: assets/doors/db0004_bifold/door_minimal.urdf (robot description, URDF)
Before this commit: robot db0004_bifold_minimal, 3 links, 2 joints
Links:
- link panel_0_0: mass 7.098194 -> 7.061165; geometry collision box size=0.751291 0.035 2.4; visual box size=0.751291 0.035 2.4
- link panel_0_1: mass 7.213566 -> 7.250595; geometry collision box size=0.769 0.035 2.4; collision sphere radius=0.016
- link world_env: geometry collision box size=0.019 0.145 2.455; collision box size=0.019 0.145 2.455
Joints:
- joint panel_0_0_hinge: origin xyz=-0.7325 0 0 rpy=0 0 0 -> xyz=-0.7345 0 0 rpy=0 0 0

File: assets/doors/db0004_bifold/door_simple.urdf (robot description, URDF)
Before this commit: robot db0004_bifold_simple, 3 links, 2 joints
Links:
- link panel_0_0: mass 7.098194 -> 7.061165; geometry collision box size=0.751291 0.035 2.4; visual box size=0.751291 0.035 2.4
- link panel_0_1: mass 7.213566 -> 7.250595; geometry collision box size=0.769 0.035 2.4; collision sphere radius=0.016
- link world_env: geometry collision box size=0.019 0.145 2.455; collision box size=0.019 0.145 2.455
Joints:
- joint panel_0_0_hinge: origin xyz=-0.7325 0 0 rpy=0 0 0 -> xyz=-0.7345 0 0 rpy=0 0 0

File: assets/doors/db0006_gate_swing/door.urdf (robot description, URDF)
Before this commit: robot db0006_gate_swing_full, 3 links, 2 joints
Joints:
- joint leaf_hinge: origin xyz=-2.403 -0.0295 0 rpy=0 0 0 -> xyz=-2.403 -0.05 0 rpy=0 0 0
- joint leaf_slide_bolt_slide: origin xyz=4.8 -0.0365 1 rpy=0 0 0 -> xyz=4.8 -0.016 1 rpy=0 0 0

File: assets/doors/db0006_gate_swing/door_minimal.urdf (robot description, URDF)
Before this commit: robot db0006_gate_swing_minimal, 3 links, 2 joints
Joints:
- joint leaf_hinge: origin xyz=-2.403 -0.0295 0 rpy=0 0 0 -> xyz=-2.403 -0.05 0 rpy=0 0 0
- joint leaf_slide_bolt_slide: origin xyz=4.8 -0.0365 1 rpy=0 0 0 -> xyz=4.8 -0.016 1 rpy=0 0 0

File: assets/doors/db0006_gate_swing/door_simple.urdf (robot description, URDF)
Before this commit: robot db0006_gate_swing_simple, 3 links, 2 joints
Joints:
- joint leaf_hinge: origin xyz=-2.403 -0.0295 0 rpy=0 0 0 -> xyz=-2.403 -0.05 0 rpy=0 0 0
- joint leaf_slide_bolt_slide: origin xyz=4.8 -0.0365 1 rpy=0 0 0 -> xyz=4.8 -0.016 1 rpy=0 0 0

File: assets/doors/db0008_sliding_bypass/door.urdf (robot description, URDF)
Before this commit: robot db0008_sliding_bypass_full, 4 links, 3 joints
Joints:
- joint leaf_0_slide: limit lower=0 upper=1.189 effort=5000 velocity=10 -> lower=0 upper=2.362 effort=5000 velocity=10; origin xyz=-1.194 -0.056 0 rpy=0 0 0 -> xyz=-1.191 -0.056 0 rpy=0 0 0
- joint leaf_1_slide: limit lower=-1.189 upper=1.189 effort=5000 velocity=10 -> lower=0 upper=1.171 effort=5000 velocity=10; origin xyz=-0.005 0 0 rpy=0 0 0 -> xyz=0 0 0 rpy=0 0 0
- joint leaf_2_slide: limit lower=0 upper=1.189 effort=5000 velocity=10 -> lower=0 upper=2.362 effort=5000 velocity=10; origin xyz=1.184 0.056 0 rpy=0 0 0 -> xyz=1.191 0.056 0 rpy=0 0 0

File: assets/doors/db0008_sliding_bypass/door_minimal.urdf (robot description, URDF)
Before this commit: robot db0008_sliding_bypass_minimal, 4 links, 3 joints
Joints:
- joint leaf_0_slide: limit lower=0 upper=1.189 effort=5000 velocity=10 -> lower=0 upper=2.362 effort=5000 velocity=10; origin xyz=-1.194 -0.056 0 rpy=0 0 0 -> xyz=-1.191 -0.056 0 rpy=0 0 0
- joint leaf_1_slide: limit lower=-1.189 upper=1.189 effort=5000 velocity=10 -> lower=0 upper=1.171 effort=5000 velocity=10; origin xyz=-0.005 0 0 rpy=0 0 0 -> xyz=0 0 0 rpy=0 0 0
- joint leaf_2_slide: limit lower=0 upper=1.189 effort=5000 velocity=10 -> lower=0 upper=2.362 effort=5000 velocity=10; origin xyz=1.184 0.056 0 rpy=0 0 0 -> xyz=1.191 0.056 0 rpy=0 0 0

File: assets/doors/db0008_sliding_bypass/door_simple.urdf (robot description, URDF)
Before this commit: robot db0008_sliding_bypass_simple, 4 links, 3 joints
Joints:
- joint leaf_0_slide: limit lower=0 upper=1.189 effort=5000 velocity=10 -> lower=0 upper=2.362 effort=5000 velocity=10; origin xyz=-1.194 -0.056 0 rpy=0 0 0 -> xyz=-1.191 -0.056 0 rpy=0 0 0
- joint leaf_1_slide: limit lower=-1.189 upper=1.189 effort=5000 velocity=10 -> lower=0 upper=1.171 effort=5000 velocity=10; origin xyz=-0.005 0 0 rpy=0 0 0 -> xyz=0 0 0 rpy=0 0 0
- joint leaf_2_slide: limit lower=0 upper=1.189 effort=5000 velocity=10 -> lower=0 upper=2.362 effort=5000 velocity=10; origin xyz=1.184 0.056 0 rpy=0 0 0 -> xyz=1.191 0.056 0 rpy=0 0 0

File: assets/doors/db0009_bifold/door.urdf (robot description, URDF)
Before this commit: robot db0009_bifold_full, 5 links, 4 joints
Links:
- link panel_0_0: mass 1.36296 -> 1.336074; geometry collision box size=0.179291 0.035 2.032; visual box size=0.179291 0.035 2.032
- link panel_0_1: mass 1.4546 -> 1.481486; geometry collision box size=0.196528 0.035 2.032; collision sphere radius=0.016
- link panel_1_0: mass 1.36296 -> 1.336074; geometry collision box size=0.179291 0.035 2.032; visual box size=0.179291 0.035 2.032
- link panel_1_1: mass 1.4546 -> 1.481486; geometry collision box size=0.196528 0.035 2.032; collision sphere radius=0.016
- link world_env: geometry collision box size=0.019 0.145 2.087; collision box size=0.019 0.145 2.087
Joints:
- joint panel_0_0_hinge: origin xyz=-0.356 0 0 rpy=0 0 0 -> xyz=-0.3595 0 0 rpy=0 0 0
- joint panel_1_0_hinge: origin xyz=0.356 0 0 rpy=0 0 0 -> xyz=0.3595 0 0 rpy=0 0 0

File: assets/doors/db0009_bifold/door_minimal.urdf (robot description, URDF)
Before this commit: robot db0009_bifold_minimal, 5 links, 4 joints
Links:
- link panel_0_0: mass 1.36296 -> 1.336074; geometry collision box size=0.179291 0.035 2.032; visual box size=0.179291 0.035 2.032
- link panel_0_1: mass 1.4546 -> 1.481486; geometry collision box size=0.196528 0.035 2.032; collision sphere radius=0.016
- link panel_1_0: mass 1.36296 -> 1.336074; geometry collision box size=0.179291 0.035 2.032; visual box size=0.179291 0.035 2.032
- link panel_1_1: mass 1.4546 -> 1.481486; geometry collision box size=0.196528 0.035 2.032; collision sphere radius=0.016
- link world_env: geometry collision box size=0.019 0.145 2.087; collision box size=0.019 0.145 2.087
Joints:
- joint panel_0_0_hinge: origin xyz=-0.356 0 0 rpy=0 0 0 -> xyz=-0.3595 0 0 rpy=0 0 0
- joint panel_1_0_hinge: origin xyz=0.356 0 0 rpy=0 0 0 -> xyz=0.3595 0 0 rpy=0 0 0

File: assets/doors/db0009_bifold/door_simple.urdf (robot description, URDF)
Before this commit: robot db0009_bifold_simple, 5 links, 4 joints
Links:
- link panel_0_0: mass 1.36296 -> 1.336074; geometry collision box size=0.179291 0.035 2.032; visual box size=0.179291 0.035 2.032
- link panel_0_1: mass 1.4546 -> 1.481486; geometry collision box size=0.196528 0.035 2.032; collision sphere radius=0.016
- link panel_1_0: mass 1.36296 -> 1.336074; geometry collision box size=0.179291 0.035 2.032; visual box size=0.179291 0.035 2.032
- link panel_1_1: mass 1.4546 -> 1.481486; geometry collision box size=0.196528 0.035 2.032; collision sphere radius=0.016
- link world_env: geometry collision box size=0.019 0.145 2.087; collision box size=0.019 0.145 2.087
Joints:
- joint panel_0_0_hinge: origin xyz=-0.356 0 0 rpy=0 0 0 -> xyz=-0.3595 0 0 rpy=0 0 0
- joint panel_1_0_hinge: origin xyz=0.356 0 0 rpy=0 0 0 -> xyz=0.3595 0 0 rpy=0 0 0

File: assets/doors/db0011_automatic_swing/door.urdf (robot description, URDF)
Before this commit: robot db0011_automatic_swing_full, 6 links, 5 joints
Links:
- link world_env: geometry collision box size=0.03 0.006 0.031; collision box size=0.045 0.3 2.147

File: assets/doors/db0011_automatic_swing/door_minimal.urdf (robot description, URDF)
Before this commit: robot db0011_automatic_swing_minimal, 4 links, 3 joints
Links:
- link world_env: geometry collision box size=0.03 0.006 0.031; collision box size=0.045 0.3 2.147
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
Commit message: Door-defect round 4: attachment gate (642/1000 doors had a part attached to nothing), ship dogs all actuate and hold, operator spring return, keypad codes physically enforced; regenerate
Co-Authored-By: Claude Opus 5 <noreply@anthropic.com>

File: assets/doors/db0001_rollup/door.urdf (robot description, URDF)
Before this commit: robot db0001_rollup_full, 2 links, 1 joints
Links:
- link curtain: geometry collision box size=0.2 0.012 0.03; collision box size=2.44 0.003 2.44
- link world_env: geometry collision box size=0.06 0.05 2.49; collision box size=0.06 0.05 2.49

File: assets/doors/db0001_rollup/door_minimal.urdf (robot description, URDF)
Before this commit: robot db0001_rollup_minimal, 2 links, 1 joints
Links:
- link curtain: geometry collision box size=0.2 0.012 0.03; collision box size=2.44 0.003 2.44

File: assets/doors/db0001_rollup/door_simple.urdf (robot description, URDF)
Before this commit: robot db0001_rollup_simple, 2 links, 1 joints
Links:
- link curtain: geometry collision box size=0.2 0.012 0.03; collision box size=2.44 0.003 2.44
- link world_env: geometry collision box size=0.06 0.05 2.49; collision box size=0.06 0.05 2.49

File: assets/doors/db0002_swing_single/door.urdf (robot description, URDF)
Before this commit: robot db0002_swing_single_full, 5 links, 4 joints
Links:
- link leaf: mass 11.329802 -> 11.141915
- link leaf_handle: mass 1.127981 -> 1.143961; geometry collision cylinder length=0.024 radius=0.011; collision cylinder length=0.024 radius=0.011
- link leaf_riser: mass 0.002104 -> 0.174012; geometry visual cylinder length=0.036 radius=0.014

File: assets/doors/db0002_swing_single/door_minimal.urdf (robot description, URDF)
Before this commit: robot db0002_swing_single_minimal, 5 links, 4 joints
Links:
- link leaf: mass 11.329802 -> 11.141915

File: assets/doors/db0002_swing_single/door_simple.urdf (robot description, URDF)
Before this commit: robot db0002_swing_single_simple, 5 links, 4 joints
Links:
- link leaf: mass 11.329802 -> 11.141915

File: assets/doors/db0003_cold_storage/door.urdf (robot description, URDF)
Before this commit: robot db0003_cold_storage_full, 5 links, 4 joints
Links:
- link leaf: mass 43.850003 -> 43.662116
- link leaf_handle: mass 2.971846 -> 2.987827; geometry collision cylinder length=0.044 radius=0.012; collision cylinder length=0.044 radius=0.012
- link leaf_riser: mass 0.002104 -> 0.174012; geometry visual cylinder length=0.036 radius=0.014
- link world_env: geometry collision box size=0.011 0.032 2.15; collision box size=0.011 0.032 2.15

File: assets/doors/db0003_cold_storage/door_minimal.urdf (robot description, URDF)
Before this commit: robot db0003_cold_storage_minimal, 5 links, 4 joints
Links:
- link leaf: mass 43.850003 -> 43.662116

File: assets/doors/db0003_cold_storage/door_simple.urdf (robot description, URDF)
Before this commit: robot db0003_cold_storage_simple, 5 links, 4 joints
Links:
- link leaf: mass 43.850003 -> 43.662116
- link world_env: geometry collision box size=0.011 0.032 2.15; collision box size=0.011 0.032 2.15

File: assets/doors/db0004_bifold/door.urdf (robot description, URDF)
Before this commit: robot db0004_bifold_full, 3 links, 2 joints
Links:
- link panel_0_0: mass 7.061165 -> 7.060608; geometry collision box size=0.751291 0.035 2.4; visual box size=0.571291 0.004 0.05292
- link panel_0_1: mass 7.250595 -> 7.251152; geometry collision box size=0.769 0.035 2.4; collision sphere radius=0.016

File: assets/doors/db0004_bifold/door_minimal.urdf (robot description, URDF)
Before this commit: robot db0004_bifold_minimal, 3 links, 2 joints
Links:
- link panel_0_0: mass 7.061165 -> 7.060608
- link panel_0_1: mass 7.250595 -> 7.251152; geometry collision box size=0.769 0.035 2.4; collision sphere radius=0.016

File: assets/doors/db0004_bifold/door_simple.urdf (robot description, URDF)
Before this commit: robot db0004_bifold_simple, 3 links, 2 joints
Links:
- link panel_0_0: mass 7.061165 -> 7.060608; geometry collision box size=0.751291 0.035 2.4; visual box size=0.751291 0.035 2.4
- link panel_0_1: mass 7.250595 -> 7.251152; geometry collision box size=0.769 0.035 2.4; collision sphere radius=0.016

File: assets/doors/db0006_gate_swing/door.urdf (robot description, URDF)
Before this commit: robot db0006_gate_swing_full, 3 links, 2 joints
Links:
- link leaf: geometry collision box size=4.8 0.045 1.2; visual box size=0.012 0.004 0.0605
- link world_env: geometry collision box size=0.014 0.005 0.034; collision box size=0.014 0.005 0.034

File: assets/doors/db0006_gate_swing/door_simple.urdf (robot description, URDF)
Before this commit: robot db0006_gate_swing_simple, 3 links, 2 joints
Links:
- link leaf: geometry collision box size=4.8 0.045 1.2; visual box size=0.012 0.004 0.0605
- link world_env: geometry collision box size=0.014 0.005 0.034; collision box size=0.014 0.005 0.034

File: assets/doors/db0009_bifold/door.urdf (robot description, URDF)
Before this commit: robot db0009_bifold_full, 5 links, 4 joints
Links:
- link panel_0_0: mass 1.336074 -> 1.335551; geometry collision box size=0.179291 0.035 2.032; visual box size=0.179291 0.035 2.032
- link panel_0_1: mass 1.481486 -> 1.482009; geometry collision box size=0.196528 0.035 2.032; collision sphere radius=0.016
- link panel_1_0: mass 1.336074 -> 1.335551; geometry collision box size=0.179291 0.035 2.032; visual box size=0.179291 0.035 2.032
- link panel_1_1: mass 1.481486 -> 1.482009; geometry collision box size=0.196528 0.035 2.032; collision sphere radius=0.016

File: assets/doors/db0009_bifold/door_minimal.urdf (robot description, URDF)
Before this commit: robot db0009_bifold_minimal, 5 links, 4 joints
Links:
- link panel_0_0: mass 1.336074 -> 1.335551
- link panel_0_1: mass 1.481486 -> 1.482009; geometry collision box size=0.196528 0.035 2.032; collision sphere radius=0.016
- link panel_1_0: mass 1.336074 -> 1.335551
- link panel_1_1: mass 1.481486 -> 1.482009; geometry collision box size=0.196528 0.035 2.032; collision sphere radius=0.016

File: assets/doors/db0009_bifold/door_simple.urdf (robot description, URDF)
Before this commit: robot db0009_bifold_simple, 5 links, 4 joints
Links:
- link panel_0_0: mass 1.336074 -> 1.335551; geometry collision box size=0.179291 0.035 2.032; visual box size=0.179291 0.035 2.032
- link panel_0_1: mass 1.481486 -> 1.482009; geometry collision box size=0.196528 0.035 2.032; collision sphere radius=0.016
- link panel_1_0: mass 1.336074 -> 1.335551; geometry collision box size=0.179291 0.035 2.032; visual box size=0.179291 0.035 2.032
- link panel_1_1: mass 1.481486 -> 1.482009; geometry collision box size=0.196528 0.035 2.032; collision sphere radius=0.016

File: assets/doors/db0010_swing_double/door.urdf (robot description, URDF)
Before this commit: robot db0010_swing_double_full, 3 links, 2 joints
Links:
- link world_env: geometry collision box size=0.019 0.145 2.147; collision box size=0.019 0.145 2.147

File: assets/doors/db0010_swing_double/door_minimal.urdf (robot description, URDF)
Before this commit: robot db0010_swing_double_minimal, 3 links, 2 joints
Links:
- link world_env: geometry collision box size=0.019 0.145 2.147; collision box size=0.019 0.145 2.147

File: assets/doors/db0010_swing_double/door_simple.urdf (robot description, URDF)
Before this commit: robot db0010_swing_double_simple, 3 links, 2 joints
Links:
- link world_env: geometry collision box size=0.019 0.145 2.147; collision box size=0.019 0.145 2.147
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