Commit message: Vision review (122 doors, 142 findings none of which any gate caught) + parity round 4 badges (925/1000 strict full, 935 doors ok)
Co-Authored-By: Claude Opus 5 <noreply@anthropic.com>

File: assets/doors/db0012_swing_single/door.urdf (robot description, URDF)
Before this commit: robot db0012_swing_single_full, 5 links, 4 joints
Links:
- link leaf: geometry collision box size=0.24 0.08 0.06; collision box size=0.813 0.006 2.134

File: assets/doors/db0040_swing_single/door.urdf (robot description, URDF)
Before this commit: robot db0040_swing_single_full, 5 links, 4 joints
Links:
- link leaf: geometry collision box size=0.914 0.035 2.134; visual box size=0.0012 0.028 0.0566

File: assets/doors/db0081_swing_single/door.urdf (robot description, URDF)
Before this commit: robot db0081_swing_single_full, 4 links, 3 joints
Links:
- link leaf: geometry collision box size=0.813 0.035 2.032; visual box size=0.0012 0.0247 0.0534

File: assets/doors/db0086_swing_single/door.urdf (robot description, URDF)
Before this commit: robot db0086_swing_single_full, 16 links, 15 joints
Links:
- link world_env: geometry collision box size=0.011 0.032 2.045; collision box size=0.011 0.032 2.045

File: assets/doors/db0101_swing_single/door.urdf (robot description, URDF)
Before this commit: robot db0101_swing_single_full, 3 links, 2 joints
Links:
- link world_env: geometry collision box size=0.011 0.032 2.451; collision box size=0.011 0.032 2.451

File: assets/doors/db0229_swing_single/door.urdf (robot description, URDF)
Before this commit: robot db0229_swing_single_full, 5 links, 4 joints
Links:
- link leaf: geometry collision box size=0.914 0.035 2.032; visual box size=0.0012 0.0247 0.0534

File: assets/doors/db0232_swing_single/door.urdf (robot description, URDF)
Before this commit: robot db0232_swing_single_full, 6 links, 5 joints
Links:
- link leaf: geometry collision box size=0.29 0.1 0.07; collision box size=0.914 0.006 2.43

File: assets/doors/db0233_swing_single/door.urdf (robot description, URDF)
Before this commit: robot db0233_swing_single_full, 16 links, 15 joints
Links:
- link world_env: geometry collision box size=0.011 0.032 2.147; collision box size=0.011 0.032 2.147

File: assets/doors/db0244_swing_single/door.urdf (robot description, URDF)
Before this commit: robot db0244_swing_single_full, 4 links, 3 joints
Links:
- link leaf: geometry collision box size=0.66 0.035 2.032; visual box size=0.0012 0.0247 0.0534

File: assets/doors/db0305_swing_single/door.urdf (robot description, URDF)
Before this commit: robot db0305_swing_single_full, 3 links, 2 joints
Links:
- link leaf: geometry collision box size=1.067 0.044 2.438; visual box size=0.024 0.004 0.274

File: assets/doors/db0348_swing_single/door.urdf (robot description, URDF)
Before this commit: robot db0348_swing_single_full, 4 links, 3 joints
Links:
- link leaf: geometry collision box size=0.813 0.035 1.985; visual box size=0.0012 0.0247 0.0534

File: assets/doors/db0374_swing_single/door.urdf (robot description, URDF)
Before this commit: robot db0374_swing_single_full, 5 links, 4 joints
Links:
- link leaf: geometry collision box size=0.29 0.1 0.07; collision box size=1.067 0.035 2.126

File: assets/doors/db0376_swing_single/door.urdf (robot description, URDF)
Before this commit: robot db0376_swing_single_full, 5 links, 4 joints
Links:
- link leaf: geometry collision box size=0.711 0.044 2.1236; visual box size=0.0012 0.0247 0.0534

File: assets/doors/db0410_swing_single/door.urdf (robot description, URDF)
Before this commit: robot db0410_swing_single_full, 4 links, 3 joints
Links:
- link leaf: geometry collision box size=0.762 0.044 2.032; visual box size=0.0012 0.0247 0.0534

File: assets/doors/db0464_swing_single/door.urdf (robot description, URDF)
Before this commit: robot db0464_swing_single_full, 16 links, 15 joints
Links:
- link world_env: geometry collision box size=0.011 0.032 2.045; collision box size=0.011 0.032 2.045

File: assets/doors/db0502_swing_single/door.urdf (robot description, URDF)
Before this commit: robot db0502_swing_single_full, 5 links, 4 joints
Links:
- link leaf: geometry collision box size=0.813 0.035 2.0216; visual box size=0.0012 0.0247 0.0534

File: assets/doors/db0519_swing_single/door.urdf (robot description, URDF)
Before this commit: robot db0519_swing_single_full, 2 links, 1 joints
Links:
- link leaf: geometry collision box size=0.914 0.044 2.134; collision cylinder length=0.16 radius=0.0095

File: assets/doors/db0521_swing_single/door.urdf (robot description, URDF)
Before this commit: robot db0521_swing_single_full, 5 links, 4 joints
Links:
- link leaf: geometry collision box size=0.813 0.035 2.1236; visual box size=0.0012 0.0247 0.0534

File: assets/doors/db0578_swing_single/door.urdf (robot description, URDF)
Before this commit: robot db0578_swing_single_full, 4 links, 3 joints
Links:
- link leaf: geometry collision box size=0.66 0.035 2.032; visual box size=0.0012 0.0247 0.0534

File: assets/doors/db0582_swing_single/door.urdf (robot description, URDF)
Before this commit: robot db0582_swing_single_full, 5 links, 4 joints
Links:
- link leaf: geometry collision box size=0.29 0.1 0.07; collision box size=0.813 0.044 2.134
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