Commit message: Merge mass and kinematics fixes: multi-leaf mass contract corrected (219 doors were 2-8x too light), releasable locks modelled as constraints not joint ranges, task_achievable + pair_swing gates
Co-Authored-By: Claude Opus 5 <noreply@anthropic.com>

File: assets/doors/db0002_swing_single/door.urdf (robot description, URDF)
Before this commit: robot db0002_swing_single_full, 5 links, 4 joints
Links:
- link leaf: mass 11.141915 -> 11.261915

File: assets/doors/db0002_swing_single/door_minimal.urdf (robot description, URDF)
Before this commit: robot db0002_swing_single_minimal, 5 links, 4 joints
Links:
- link leaf: mass 11.141915 -> 11.261915

File: assets/doors/db0002_swing_single/door_simple.urdf (robot description, URDF)
Before this commit: robot db0002_swing_single_simple, 5 links, 4 joints
Links:
- link leaf: mass 11.141915 -> 11.261915

File: assets/doors/db0003_cold_storage/door.urdf (robot description, URDF)
Before this commit: robot db0003_cold_storage_full, 5 links, 4 joints
Links:
- link leaf: mass 43.662116 -> 43.742116

File: assets/doors/db0003_cold_storage/door_minimal.urdf (robot description, URDF)
Before this commit: robot db0003_cold_storage_minimal, 5 links, 4 joints
Links:
- link leaf: mass 43.662116 -> 43.742116

File: assets/doors/db0003_cold_storage/door_simple.urdf (robot description, URDF)
Before this commit: robot db0003_cold_storage_simple, 5 links, 4 joints
Links:
- link leaf: mass 43.662116 -> 43.742116

File: assets/doors/db0004_bifold/door.urdf (robot description, URDF)
Before this commit: robot db0004_bifold_full, 3 links, 2 joints
Links:
- link panel_0_0: mass 7.060608 -> 14.037347
- link panel_0_1: mass 7.251152 -> 14.416173

File: assets/doors/db0004_bifold/door_minimal.urdf (robot description, URDF)
Before this commit: robot db0004_bifold_minimal, 3 links, 2 joints
Links:
- link panel_0_0: mass 7.060608 -> 14.037347
- link panel_0_1: mass 7.251152 -> 14.416173

File: assets/doors/db0004_bifold/door_simple.urdf (robot description, URDF)
Before this commit: robot db0004_bifold_simple, 3 links, 2 joints
Links:
- link panel_0_0: mass 7.060608 -> 14.037347
- link panel_0_1: mass 7.251152 -> 14.416173

File: assets/doors/db0006_gate_swing/door.urdf (robot description, URDF)
Before this commit: robot db0006_gate_swing_full, 3 links, 2 joints
Links:
- link leaf: mass 76.756275 -> 78.356275

File: assets/doors/db0006_gate_swing/door_minimal.urdf (robot description, URDF)
Before this commit: robot db0006_gate_swing_minimal, 3 links, 2 joints
Links:
- link leaf: mass 76.756275 -> 78.356275

File: assets/doors/db0006_gate_swing/door_simple.urdf (robot description, URDF)
Before this commit: robot db0006_gate_swing_simple, 3 links, 2 joints
Links:
- link leaf: mass 76.756275 -> 78.356275

File: assets/doors/db0008_sliding_bypass/door.urdf (robot description, URDF)
Before this commit: robot db0008_sliding_bypass_full, 4 links, 3 joints
Links:
- link leaf_0: mass 12.401707 -> 37.171787
- link leaf_1: mass 12.401707 -> 37.171787
- link leaf_2: mass 12.401707 -> 37.171787

File: assets/doors/db0008_sliding_bypass/door_minimal.urdf (robot description, URDF)
Before this commit: robot db0008_sliding_bypass_minimal, 4 links, 3 joints
Links:
- link leaf_0: mass 12.401707 -> 37.171787
- link leaf_1: mass 12.401707 -> 37.171787
- link leaf_2: mass 12.401707 -> 37.171787

File: assets/doors/db0008_sliding_bypass/door_simple.urdf (robot description, URDF)
Before this commit: robot db0008_sliding_bypass_simple, 4 links, 3 joints
Links:
- link leaf_0: mass 12.401707 -> 37.171787
- link leaf_1: mass 12.401707 -> 37.171787
- link leaf_2: mass 12.401707 -> 37.171787

File: assets/doors/db0009_bifold/door.urdf (robot description, URDF)
Before this commit: robot db0009_bifold_full, 5 links, 4 joints
Links:
- link panel_0_0: mass 1.335551 -> 5.178672
- link panel_0_1: mass 1.482009 -> 5.746568
- link panel_1_0: mass 1.335551 -> 5.178672
- link panel_1_1: mass 1.482009 -> 5.746568

File: assets/doors/db0009_bifold/door_minimal.urdf (robot description, URDF)
Before this commit: robot db0009_bifold_minimal, 5 links, 4 joints
Links:
- link panel_0_0: mass 1.335551 -> 5.178672
- link panel_0_1: mass 1.482009 -> 5.746568
- link panel_1_0: mass 1.335551 -> 5.178672
- link panel_1_1: mass 1.482009 -> 5.746568

File: assets/doors/db0009_bifold/door_simple.urdf (robot description, URDF)
Before this commit: robot db0009_bifold_simple, 5 links, 4 joints
Links:
- link panel_0_0: mass 1.335551 -> 5.178672
- link panel_0_1: mass 1.482009 -> 5.746568
- link panel_1_0: mass 1.335551 -> 5.178672
- link panel_1_1: mass 1.482009 -> 5.746568

File: assets/doors/db0010_swing_double/door.urdf (robot description, URDF)
Before this commit: robot db0010_swing_double_full, 3 links, 2 joints
Links:
- link leaf_a: mass 50.839121 -> 98.253242
- link leaf_b: mass 50.839121 -> 98.253242

File: assets/doors/db0010_swing_double/door_minimal.urdf (robot description, URDF)
Before this commit: robot db0010_swing_double_minimal, 3 links, 2 joints
Links:
- link leaf_a: mass 50.839121 -> 98.253242
- link leaf_b: mass 50.839121 -> 98.253242
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